Commit message: update orientations of joints to match actual robot

File: urdf/smaldog.urdf (robot description, URDF)
Before this commit: robot SMALdog, 13 links, 12 joints
Links:
- link lf_tibia_link: geometry visual cylinder length=0.086 radius=0.00635
- link lr_tibia_link: geometry visual cylinder length=0.086 radius=0.00635
- link rf_tibia_link: geometry visual cylinder length=0.086 radius=0.00635
- link rr_tibia_link: geometry visual cylinder length=0.086 radius=0.00635
Joints:
- joint lf_tibia_joint: axis 0 1 0 -> 0 -1 0
- joint lr_femur_joint: axis 0 1 0 -> 0 -1 0
- joint rf_coxa_joint: axis 1 0 0 -> -1 0 0
- joint rf_tibia_joint: axis 0 1 0 -> 0 -1 0
- joint rr_coxa_joint: axis 1 0 0 -> -1 0 0
- joint rr_femur_joint: axis 0 1 0 -> 0 -1 0

Commit message: a bit more urdf

File: urdf/smaldog.urdf (robot description, URDF)
Before this commit: robot SMALdog, 13 links, 12 joints
Links:
- link body_link: geometry visual box size=0.2 0.065 0.055
- link lf_coxa_link: geometry visual cylinder length=0.050 radius=0.00635
- link lf_femur_link: geometry visual cylinder length=0.064 radius=0.01
- link lr_coxa_link: geometry visual cylinder length=0.050 radius=0.00635
- link lr_femur_link: geometry visual cylinder length=0.064 radius=0.01
- link rf_coxa_link: geometry visual cylinder length=0.050 radius=0.00635
- link rf_femur_link: geometry visual cylinder length=0.064 radius=0.01
- link rr_coxa_link: geometry visual cylinder length=0.050 radius=0.00635
- link rr_femur_link: geometry visual cylinder length=0.064 radius=0.01

Commit message: update urdf joint names

File: urdf/smaldog.urdf (robot description, URDF)
Before this commit: robot SMALdog, 13 links, 12 joints
Links:
- removed link lf_coxa_link
- removed link lr_coxa_link
- removed link rf_coxa_link
- removed link rr_coxa_link
- added link lf_shoulder_link; visual cylinder length=0.050 radius=0.00635
- added link lr_shoulder_link; visual cylinder length=0.050 radius=0.00635
- added link rf_shoulder_link; visual cylinder length=0.050 radius=0.00635
- added link rr_shoulder_link; visual cylinder length=0.050 radius=0.00635
Joints:
- removed joint lf_coxa_joint
- removed joint lf_femur_joint
- removed joint lf_tibia_joint
- removed joint lr_coxa_joint
- removed joint lr_femur_joint
- removed joint lr_tibia_joint
- removed joint rf_coxa_joint
- removed joint rf_femur_joint
- removed joint rf_tibia_joint
- removed joint rr_coxa_joint
- removed joint rr_femur_joint
- removed joint rr_tibia_joint
- added joint lf_flex_joint: type revolute, parent lf_shoulder_link, child lf_femur_link, origin xyz=0 0.050 0 rpy=0 0 0, axis 0 1 0, limit lower=-1.57 upper=1.57 effort=30 velocity=0.5
- added joint lf_knee_joint: type revolute, parent lf_femur_link, child lf_tibia_link, origin xyz=0 0 -0.064 rpy=0 0 0, axis 0 -1 0, limit lower=-1.57 upper=1.57 effort=30 velocity=0.5
- added joint lf_pitch_joint: type revolute, parent body_link, child lf_shoulder_link, origin xyz=0.086 0.019 0 rpy=0 0 0, axis 1 0 0, limit lower=-1.57 upper=1.57 effort=30 velocity=0.5
- added joint lr_flex_joint: type revolute, parent lr_shoulder_link, child lr_femur_link, origin xyz=0 0.050 0 rpy=0 0 0, axis 0 -1 0, limit lower=-1.57 upper=1.57 effort=30 velocity=0.5
- added joint lr_knee_joint: type revolute, parent lr_femur_link, child lr_tibia_link, origin xyz=0 0 -0.064 rpy=0 0 0, axis 0 1 0, limit lower=-1.57 upper=1.57 effort=30 velocity=0.5
- added joint lr_pitch_joint: type revolute, parent body_link, child lr_shoulder_link, origin xyz=-0.086 0.019 0 rpy=0 0 0, axis 1 0 0, limit lower=-1.57 upper=1.57 effort=30 velocity=0.5
- added joint rf_flex_joint: type revolute, parent rf_shoulder_link, child rf_femur_link, origin xyz=0 -0.050 0 rpy=0 0 0, axis 0 1 0, limit lower=-1.57 upper=1.57 effort=30 velocity=0.5
- added joint rf_knee_joint: type revolute, parent rf_femur_link, child rf_tibia_link, origin xyz=0 0 -0.064 rpy=0 0 0, axis 0 -1 0, limit lower=-1.57 upper=1.57 effort=30 velocity=0.5
- added joint rf_pitch_joint: type revolute, parent body_link, child rf_shoulder_link, origin xyz=0.086 -0.019 0 rpy=0 0 0, axis -1 0 0, limit lower=-1.57 upper=1.57 effort=30 velocity=0.5
- added joint rr_flex_joint: type revolute, parent rr_shoulder_link, child rr_femur_link, origin xyz=0 -0.050 0 rpy=0 0 0, axis 0 -1 0, limit lower=-1.57 upper=1.57 effort=30 velocity=0.5
- added joint rr_knee_joint: type revolute, parent rr_femur_link, child rr_tibia_link, origin xyz=0 0 -0.064 rpy=0 0 0, axis 0 1 0, limit lower=-1.57 upper=1.57 effort=30 velocity=0.5
- added joint rr_pitch_joint: type revolute, parent body_link, child rr_shoulder_link, origin xyz=-0.086 -0.019 0 rpy=0 0 0, axis -1 0 0, limit lower=-1.57 upper=1.57 effort=30 velocity=0.5

Commit message: make all joints a right-handed system, hacks to leg_ik, create stand up test script

File: urdf/smaldog.urdf (robot description, URDF)
Before this commit: robot SMALdog, 13 links, 12 joints
Joints:
- joint lf_flex_joint: limit lower=-1.57 upper=1.57 effort=30 velocity=0.5 -> lower=-1.2629 upper=2.2549 effort=1.1767 velocity=6.17846
- joint lf_knee_joint: axis 0 -1 0 -> 0 1 0; limit lower=-1.57 upper=1.57 effort=30 velocity=0.5 -> lower=-2.807 upper=0.588 effort=1.1767 velocity=6.17846
- joint lf_pitch_joint: limit lower=-1.57 upper=1.57 effort=30 velocity=0.5 -> lower=-0.3221 upper=1.0 effort=1.1767 velocity=6.17846
- joint lr_flex_joint: axis 0 -1 0 -> 0 1 0; limit lower=-1.57 upper=1.57 effort=30 velocity=0.5 -> lower=-2.2549 upper=1.2629 effort=1.1767 velocity=6.17846
- joint lr_knee_joint: limit lower=-1.57 upper=1.57 effort=30 velocity=0.5 -> lower=-0.588 upper=2.807 effort=1.1767 velocity=6.17846
- joint lr_pitch_joint: limit lower=-1.57 upper=1.57 effort=30 velocity=0.5 -> lower=-0.3221 upper=1.0 effort=1.1767 velocity=6.17846
- joint rf_flex_joint: limit lower=-1.57 upper=1.57 effort=30 velocity=0.5 -> lower=-1.2629 upper=2.2549 effort=1.1767 velocity=6.17846
- joint rf_knee_joint: axis 0 -1 0 -> 0 1 0; limit lower=-1.57 upper=1.57 effort=30 velocity=0.5 -> lower=-2.807 upper=0.588 effort=1.1767 velocity=6.17846
- joint rf_pitch_joint: axis -1 0 0 -> 1 0 0; limit lower=-1.57 upper=1.57 effort=30 velocity=0.5 -> lower=-1.0 upper=0.3221 effort=1.1767 velocity=6.17846
- joint rr_flex_joint: axis 0 -1 0 -> 0 1 0; limit lower=-1.57 upper=1.57 effort=30 velocity=0.5 -> lower=-2.2549 upper=1.2629 effort=1.1767 velocity=6.17846
- joint rr_knee_joint: limit lower=-1.57 upper=1.57 effort=30 velocity=0.5 -> lower=-0.588 upper=2.807 effort=1.1767 velocity=6.17846
- joint rr_pitch_joint: axis -1 0 0 -> 1 0 0; limit lower=-1.57 upper=1.57 effort=30 velocity=0.5 -> lower=-1.0 upper=0.3221 effort=1.1767 velocity=6.17846
